Commit message: clean up

File: agents/iris/iris.xacro (robot description, xacro)
@@ -4,6 +4,5 @@
   <xacro:property name="ns" value="iris" />
   <xacro:property name="mesh_root" value="package://ardupilot_sim/agents/iris/meshes" />
-  <!-- <xacro:property name="mesh_root" value="package://iris/meshes" /> -->
-  <xacro:property name="mass" value="1.75" /> <!-- [kg] -->
+  <xacro:property name="mass" value="1.5" /> <!-- [kg] -->
   <xacro:property name="body_inertia">
     <inertia ixx="0.008" ixy="0.0" ixz="0.0" iyy="0.0815" iyz="0.0" izz="0.017" />
@@ -45,4 +44,5 @@
     <material>Gazebo/DarkGrey</material>
   </gazebo>
+  <!-- *********************** GAZEBO ROBOT PLUGINS ******************* -->
   <xacro:include filename="$(find ardupilot_sim)/xacro/imu.xacro" />
   <xacro:imu ns="${ns}" update_rate="1000">
@@ -62,7 +62,4 @@
     <origin xyz="-0.13 -0.2 0.023" rpy="0 0 0" />
   </xacro:rotor>
-<!--   <gazebo reference="${ns}/base_link">
-    <material>Gazebo/FlatBlack</material>
-  </gazebo> -->
   <xacro:include filename="$(find ardupilot_sim)/xacro/arducopter.xacro" />
   <xacro:arducopter ns="${ns}" />

Commit message: initial commit for plane sitl

File: agents/iris/iris.xacro (robot description, xacro)
@@ -9,4 +9,5 @@
   </xacro:property>
   <xacro:property name="rotor_inertia">
+    <mass value="0.025"/>
     <inertia ixx="9.75e-06" ixy="0.0" ixz="0.0" iyy="0.000166704" iyz="0.0" izz="0.000167604" />
   </xacro:property>
@@ -47,18 +48,19 @@
   <xacro:include filename="$(find ardupilot_sim)/xacro/imu.xacro" />
   <xacro:imu ns="${ns}" update_rate="1000">
+    <axis xyz="0 0 1"/>
     <pose>0 0 0 3.141593 0 0</pose>
   </xacro:imu>
   <xacro:include filename="$(find ardupilot_sim)/xacro/rotor.xacro" />
   <xacro:rotor ns="${ns}" motor_number="0" prop_dir="ccw">
-    <origin xyz="0.13 -0.22 0.023" rpy="0 0 0" />
+    <pose value="0.13 -0.22 0.023 0 0 0" />
   </xacro:rotor>
   <xacro:rotor ns="${ns}" motor_number="1" prop_dir="ccw">
-    <origin xyz="-0.13 0.2 0.023" rpy="0 0 0" />
+    <pose value="-0.13 0.2 0.023 0 0 0" />
   </xacro:rotor>
   <xacro:rotor ns="${ns}" motor_number="2" prop_dir="cw">
-    <origin xyz="0.13 0.22 0.023" rpy="0 0 0" />
+    <pose value="0.13 0.22 0.023 0 0 0" />
   </xacro:rotor>
   <xacro:rotor ns="${ns}" motor_number="3" prop_dir="cw">
-    <origin xyz="-0.13 -0.2 0.023" rpy="0 0 0" />
+    <pose value="-0.13 -0.2 0.023 0 0 0" />
   </xacro:rotor>
   <xacro:include filename="$(find ardupilot_sim)/xacro/arducopter.xacro" />

File: xacro/arduplane.xacro (robot description, xacro)
@@ -1,7 +1,7 @@
 <?xml version="1.0"?>
-<robot name="iris" xmlns:xacro="http://ros.org/wiki/xacro">
-  <xacro:macro name="arducopter" params="ns">
+<robot name="plane" xmlns:xacro="http://ros.org/wiki/xacro">
+  <xacro:macro name="arduplane" params="ns">
     <gazebo>
-      <plugin name="arducopter_plugin" filename="libArduPilotPlugin.so">
+      <plugin name="arduplane_plugin" filename="libArduPilotPlugin.so">
         <fdm_addr>127.0.0.1</fdm_addr>
         <fdm_port_in>9002</fdm_port_in>
@@ -37,43 +37,53 @@
         </control>
         <control channel="1">
-          <type>VELOCITY</type>
+          <type>POSITION</type>
           <offset>0</offset>
           <p_gain>0.20</p_gain>
           <i_gain>0</i_gain>
-          <d_gain>0</d_gain>
+          <d_gain>0.01</d_gain>
           <i_max>0</i_max>
           <i_min>0</i_min>
           <cmd_max>2.5</cmd_max>
           <cmd_min>-2.5</cmd_min>
-          <jointName>${ns}/rotor_1_joint</jointName>
-          <multiplier>838</multiplier>
+          <jointName>${ns}/left_aileron_joint</jointName>
           <controlVelocitySlowdownSim>1</controlVelocitySlowdownSim>
         </control>
         <control channel="2">
-          <type>VELOCITY</type>
+          <type>POSITION</type>
           <offset>0</offset>
           <p_gain>0.20</p_gain>
           <i_gain>0</i_gain>
-          <d_gain>0</d_gain>
+          <d_gain>0.01</d_gain>
           <i_max>0</i_max>
           <i_min>0</i_min>
           <cmd_max>2.5</cmd_max>
           <cmd_min>-2.5</cmd_min>
-          <jointName>${ns}/rotor_2_joint</jointName>
-          <multiplier>-838</multiplier>
+          <jointName>${ns}/right_aileron_joint</jointName>
           <controlVelocitySlowdownSim>1</controlVelocitySlowdownSim>
         </control>
         <control channel="3">
-          <type>VELOCITY</type>
+          <type>POSITION</type>
           <offset>0</offset>
           <p_gain>0.20</p_gain>
           <i_gain>0</i_gain>
-          <d_gain>0</d_gain>
+          <d_gain>0.01</d_gain>
           <i_max>0</i_max>
           <i_min>0</i_min>
           <cmd_max>2.5</cmd_max>
           <cmd_min>-2.5</cmd_min>
-          <jointName>${ns}/rotor_3_joint</jointName>
-          <multiplier>-838</multiplier>
+          <jointName>${ns}/elevator_joint</jointName>
+          <controlVelocitySlowdownSim>1</controlVelocitySlowdownSim>
+        </control>
+        <control channel="4">
+          <type>POSITION</type>
+          <offset>0</offset>
+          <p_gain>0.20</p_gain>
+          <i_gain>0</i_gain>
+          <d_gain>0.01</d_gain>
+          <i_max>0</i_max>
+          <i_min>0</i_min>
+          <cmd_max>2.5</cmd_max>
+          <cmd_min>-2.5</cmd_min>
+          <jointName>${ns}/rudder_joint</jointName>
           <controlVelocitySlowdownSim>1</controlVelocitySlowdownSim>
         </control>

File: xacro/imu.xacro (robot description, xacro)
@@ -1,5 +1,5 @@
 <?xml version="1.0"?>
 <robot xmlns:xacro="http://ros.org/wiki/xacro">
-  <xacro:macro name="imu" params="ns update_rate *pose">
+  <xacro:macro name="imu" params="ns update_rate *axis *pose">
     <link name="${ns}/imu_link">
       <inertial>
@@ -13,5 +13,5 @@
       <child link="${ns}/imu_link" />
       <origin xyz="0 0 0" rpy="0 0 0"/>
-      <axis xyz="0 0 1"/>
+      <xacro:insert_block name="axis" />
       <dynamics damping="1"/>
       <limit effort="0" velocity="0" lower="0" upper="0" />

File: xacro/rotor.xacro (robot description, xacro)
@@ -1,8 +1,9 @@
 <?xml version="1.0"?>
 <robot xmlns:xacro="http://ros.org/wiki/xacro">
-  <xacro:macro name="rotor" params="ns motor_number prop_dir *origin">
+  <xacro:macro name="rotor" params="ns motor_number prop_dir *pose">
     <link name="${ns}/rotor_${motor_number}">
+      <xacro:insert_block name="pose" />
       <inertial>
-        <mass value="0.025" />
+        <!--Look in iris.xacro or plane.xacro for definition -->
         <xacro:insert_block name="rotor_inertia" />
       </inertial>
@@ -19,5 +20,4 @@
     </link>
     <joint name="${ns}/rotor_${motor_number}_joint" type="revolute">
-      <xacro:insert_block name="origin" />
       <parent link="${ns}/base_link" />
       <child link="${ns}/rotor_${motor_number}" />

Commit message: Ardupilot is now flying a 4 channel plane (cessna) with waypoints

File: agents/iris/iris.xacro (robot description, xacro)
@@ -10,5 +10,5 @@
   <xacro:property name="rotor_inertia">
     <mass value="0.025"/>
-    <inertia ixx="9.75e-06" ixy="0.0" ixz="0.0" iyy="0.000166704" iyz="0.0" izz="0.000167604" />
+    <inertia ixx=".0003675" ixy="0.0" ixz="0.0" iyy="0.0003698" iyz="0.0" izz="0.00003187" />
   </xacro:property>
   <!-- *********************** GAZEBO ROBOT DEFINITION ******************* -->
@@ -53,14 +53,14 @@
   <xacro:include filename="$(find ardupilot_sim)/xacro/rotor.xacro" />
   <xacro:rotor ns="${ns}" motor_number="0" prop_dir="ccw">
-    <pose value="0.13 -0.22 0.023 0 0 0" />
+    <origin xyz="0.13 -0.22 0.023" rpy="0 0 0" />
   </xacro:rotor>
   <xacro:rotor ns="${ns}" motor_number="1" prop_dir="ccw">
-    <pose value="-0.13 0.2 0.023 0 0 0" />
+    <origin xyz="-0.13 0.2 0.023" rpy="0 0 0" />
   </xacro:rotor>
   <xacro:rotor ns="${ns}" motor_number="2" prop_dir="cw">
-    <pose value="0.13 0.22 0.023 0 0 0" />
+    <origin xyz="0.13 0.22 0.023" rpy="0 0 0" />
   </xacro:rotor>
   <xacro:rotor ns="${ns}" motor_number="3" prop_dir="cw">
-    <pose value="-0.13 -0.2 0.023 0 0 0" />
+    <origin xyz="-0.13 -0.2 0.023" rpy="0 0 0" />
   </xacro:rotor>
   <xacro:include filename="$(find ardupilot_sim)/xacro/arducopter.xacro" />

File: xacro/arduplane.xacro (robot description, xacro)
@@ -11,78 +11,75 @@
             Only change model and gazebo from XYZ to XY-Z coordinates
         -->
-        <modelXYZToAirplaneXForwardZDown>0 0 0 3.141593 0 0</modelXYZToAirplaneXForwardZDown>
-        <gazeboXYZToNED>0 0 0 3.141593 0 1.5708</gazeboXYZToNED>
+        <modelXYZToAirplaneXForwardZDown>0 0 0 0 0 0</modelXYZToAirplaneXForwardZDown>
+        <gazeboXYZToNED>0 0 0 3.141593 0 0</gazeboXYZToNED>
         <imuName>${ns}/imu_link::imu_sensor</imuName>
         <connectionTimeoutMaxCount>5</connectionTimeoutMaxCount>
-        <control channel="0">
-        <!--
-            incoming control command [0, 1]
-            so offset it by 0 to get [0, 1]
-            and divide max target by 1.
-            offset = 0
-            multiplier = 838 max rpm / 1 = 838
-          -->
+        <control channel="2">
           <type>VELOCITY</type>
           <offset>0</offset>
+          <p_gain>0</p_gain>
+          <i_gain>10</i_gain>
+          <d_gain>0</d_gain>
+          <i_max>100000</i_max>
+          <i_min>-100000</i_min>
+          <cmd_max>2.5</cmd_max>
+          <cmd_min>0</cmd_min>
+          <jointName>${ns}/propeller_joint</jointName>
+          <multiplier>838</multiplier>
+          <rotorVelocitySlowdownSim>1</rotorVelocitySlowdownSim>
+        </control>
+        <control channel="0">
+          <type>POSITION</type>
+          <offset>-0.5</offset>
           <p_gain>0.20</p_gain>
           <i_gain>0</i_gain>
-          <d_gain>0</d_gain>
+          <d_gain>1.50</d_gain>
           <i_max>0</i_max>
           <i_min>0</i_min>
-          <cmd_max>2.5</cmd_max>
-          <cmd_min>-2.5</cmd_min>
-          <jointName>${ns}/rotor_0_joint</jointName>
-          <multiplier>838</multiplier>
+          <cmd_max>1.0</cmd_max>
+          <cmd_min>-1.0</cmd_min>
+          <multiplier>-1</multiplier>
+          <jointName>${ns}/left_aileron_joint</jointName>
+          <controlVelocitySlowdownSim>1</controlVelocitySlowdownSim>
+        </control>
+        <control channel="0">
+          <type>POSITION</type>
+          <offset>-0.5</offset>
+          <p_gain>0.20</p_gain>
+          <i_gain>0</i_gain>
+          <d_gain>1.50</d_gain>
+          <i_max>0</i_max>
+          <i_min>0</i_min>
+          <cmd_max>1.0</cmd_max>
+          <cmd_min>-1.0</cmd_min>
+          <multiplier>1</multiplier>
+          <jointName>${ns}/right_aileron_joint</jointName>
           <controlVelocitySlowdownSim>1</controlVelocitySlowdownSim>
         </control>
         <control channel="1">
           <type>POSITION</type>
-          <offset>0</offset>
+          <offset>-0.5</offset>
           <p_gain>0.20</p_gain>
           <i_gain>0</i_gain>
-          <d_gain>0.01</d_gain>
+          <d_gain>1.50</d_gain>
           <i_max>0</i_max>
           <i_min>0</i_min>
-          <cmd_max>2.5</cmd_max>
-          <cmd_min>-2.5</cmd_min>
-          <jointName>${ns}/left_aileron_joint</jointName>
-          <controlVelocitySlowdownSim>1</controlVelocitySlowdownSim>
-        </control>
-        <control channel="2">
-          <type>POSITION</type>
-          <offset>0</offset>
-          <p_gain>0.20</p_gain>
-          <i_gain>0</i_gain>
-          <d_gain>0.01</d_gain>
-          <i_max>0</i_max>
-          <i_min>0</i_min>
-          <cmd_max>2.5</cmd_max>
-          <cmd_min>-2.5</cmd_min>
-          <jointName>${ns}/right_aileron_joint</jointName>
+          <cmd_max>1.0</cmd_max>
+          <cmd_min>-1.0</cmd_min>
+          <multiplier>1</multiplier>
+          <jointName>${ns}/elevators_joint</jointName>
           <controlVelocitySlowdownSim>1</controlVelocitySlowdownSim>
         </control>
         <control channel="3">
           <type>POSITION</type>
-          <offset>0</offset>
+          <offset>-0.5</offset>
           <p_gain>0.20</p_gain>
           <i_gain>0</i_gain>
-          <d_gain>0.01</d_gain>
+          <d_gain>1.50</d_gain>
           <i_max>0</i_max>
           <i_min>0</i_min>
-          <cmd_max>2.5</cmd_max>
-          <cmd_min>-2.5</cmd_min>
-          <jointName>${ns}/elevator_joint</jointName>
-          <controlVelocitySlowdownSim>1</controlVelocitySlowdownSim>
-        </control>
-        <control channel="4">
-          <type>POSITION</type>
-          <offset>0</offset>
-          <p_gain>0.20</p_gain>
-          <i_gain>0</i_gain>
-          <d_gain>0.01</d_gain>
-          <i_max>0</i_max>
-          <i_min>0</i_min>
-          <cmd_max>2.5</cmd_max>
-          <cmd_min>-2.5</cmd_min>
+          <cmd_max>1.0</cmd_max>
+          <cmd_min>-1.0</cmd_min>
+          <multiplier>1</multiplier>
           <jointName>${ns}/rudder_joint</jointName>
           <controlVelocitySlowdownSim>1</controlVelocitySlowdownSim>

File: xacro/control_surface.xacro (robot description, xacro)
@@ -1,39 +1,24 @@
 <?xml version="1.0"?>
 <robot xmlns:xacro="http://ros.org/wiki/xacro">
-  <xacro:macro name="control_surface" params="ns surface_name limit *pose *xyz">
+  <xacro:macro name="control_surface" params="ns surface_name limit *lorigin *vorigin *jorigin *axis">
     <link name="${ns}/${surface_name}">
       <inertial>
-        <mass value="0.000000001" />
-        <inertia>
-          <ixx>0.000001</ixx>
-          <ixy>0.0</ixy>
-          <iyy>0.000001</iyy>
-          <ixz>0.0</ixz>
-          <iyz>0.0</iyz>
-          <izz>0.000001</izz>
-        </inertia>
-        <xacro:insert_block name="pose" />
+        <mass value="0.0001" />
+        <inertia ixx="0.0038166" ixy="0" ixz="0" iyy="0.0036" iyz="0" izz="0.003816"/>
       </inertial>
+      <visual>
+        <geometry>
+          <!--mesh root comes from cessna.xacro-->
+          <mesh filename="${mesh_root}/${surface_name}.dae" scale="0.1 0.1 0.1"/>
+        </geometry>
+        <xacro:insert_block name="vorigin" />
+      </visual>
     </link>
     <joint name="${ns}/${surface_name}_joint" type="revolute">
       <parent link="${ns}/base_link" />
       <child link="${ns}/${surface_name}" />
-      <xacro:insert_block name="pose" />
-      <axis>
-        <xacro:insert_block name="xyz" />
-        <limit>
-          <!-- -30/+30 deg. -->
-          <lower>-${limit}</lower>
-          <upper>${limit}</upper>
-        </limit>
-        <dynamics>
-          <damping>1.000</damping>
-        </dynamics>
-      </axis>
-      <physics>
-        <ode>
-          <implicit_spring_damper>1</implicit_spring_damper>
-        </ode>
-      </physics>
+      <xacro:insert_block name="jorigin" />
+      <xacro:insert_block name="axis" />
+      <limit lower="${-limit}" upper="${limit}" effort="-1" velocity="-1"/>
     </joint>
     <gazebo>
@@ -41,8 +26,8 @@
         <!--Look in plane.xacro for definitions-->
         <xacro:if value="${surface_name == 'left_aileron'}">
-          <xacro:insert_block name="aileron_coeffs"/>
+          <xacro:insert_block name="left_aileron_coeffs"/>
         </xacro:if>
         <xacro:if value="${surface_name == 'right_aileron'}">
-          <xacro:insert_block name="aileron_coeffs"/>
+          <xacro:insert_block name="right_aileron_coeffs"/>
         </xacro:if>
         <xacro:if value="${surface_name == 'rudder'}">
@@ -53,6 +38,6 @@
         </xacro:if>
         <forward>1 0 0</forward>
-        <link_name>base_link</link_name>
-        <control_joint_name>${surface_name}_joint</control_joint_name>
+        <link_name>${ns}/base_link</link_name>
+        <control_joint_name>${ns}/${surface_name}_joint</control_joint_name>
       </plugin>
     </gazebo>

File: xacro/rotor.xacro (robot description, xacro)
@@ -1,7 +1,6 @@
 <?xml version="1.0"?>
 <robot xmlns:xacro="http://ros.org/wiki/xacro">
-  <xacro:macro name="rotor" params="ns motor_number prop_dir *pose">
+  <xacro:macro name="rotor" params="ns motor_number prop_dir *origin">
     <link name="${ns}/rotor_${motor_number}">
-      <xacro:insert_block name="pose" />
       <inertial>
         <!--Look in iris.xacro or plane.xacro for definition -->
@@ -20,4 +19,5 @@
     </link>
     <joint name="${ns}/rotor_${motor_number}_joint" type="revolute">
+      <xacro:insert_block name="origin" />
       <parent link="${ns}/base_link" />
       <child link="${ns}/rotor_${motor_number}" />
