Commit message: Added capability for multiple plane agents
Added params to plane_sitl to limit number of windows

fixed plane_sitl to still launch MAVProxy console

File: agents/cessna/cessna.xacro (robot description, xacro)
@@ -2,5 +2,6 @@
 <robot name="cessna" xmlns:xacro="http://ros.org/wiki/xacro">
   <!-- Properties -->
-  <xacro:property name="ns" value="cessna" />
+  <xacro:arg name="instance" default="0" />
+  <xacro:property name="ns" value="cessna_$(arg instance)" />
   <xacro:property name="mesh_root" value="package://ardupilot_sim/agents/cessna/meshes" />
   <xacro:property name="mass" value="4" /> <!-- [kg] -->
@@ -135,5 +136,5 @@
     <axis xyz="0 0 1"/>
   </xacro:control_surface>
-  <xacro:include filename="$(find ardupilot_sim)/xacro/arduplane.xacro" />
-  <xacro:arduplane ns="${ns}" />
+  <xacro:include filename="$(find ardupilot_sim)/xacro/arduplane.xacro"/>
+  <xacro:arduplane ns="${ns}" inst="$(arg instance)"/>
 </robot>

File: xacro/arduplane.xacro (robot description, xacro)
@@ -1,10 +1,10 @@
 <?xml version="1.0"?>
 <robot name="plane" xmlns:xacro="http://ros.org/wiki/xacro">
-  <xacro:macro name="arduplane" params="ns">
+  <xacro:macro name="arduplane" params="ns inst">
     <gazebo>
-      <plugin name="arduplane_plugin" filename="libArduPilotPlugin.so">
+      <plugin name="${ns}_arduplane_plugin" filename="libArduPilotPlugin.so">
         <fdm_addr>127.0.0.1</fdm_addr>
-        <fdm_port_in>9002</fdm_port_in>
-        <fdm_port_out>9003</fdm_port_out>
+        <fdm_port_in>${9002 + 10*inst} </fdm_port_in>
+        <fdm_port_out>${9003 + 10*inst}</fdm_port_out>
         <!--
             Require by APM :

Commit message: plane tuning

File: agents/cessna/cessna.xacro (robot description, xacro)
@@ -4,7 +4,7 @@
   <xacro:property name="ns" value="cessna" />
   <xacro:property name="mesh_root" value="package://ardupilot_sim/agents/cessna/meshes" />
-  <xacro:property name="mass" value="1.5" /> <!-- [kg] -->
+  <xacro:property name="mass" value="4" /> <!-- [kg] -->
   <xacro:property name="body_inertia">
-    <inertia ixx="12.85315" ixy="0.0" ixz="0.0" iyy=".1825930" iyz="0.0" izz=".002666894" />
+    <inertia ixx="0.1285315" ixy="0.0" ixz="0.0" iyy="0.1825930" iyz="0.0" izz="0.2666894" />
   </xacro:property>
   <xacro:property name="rotor_inertia">
@@ -93,6 +93,6 @@
     <minDepth>0.001</minDepth>
     <!-- Friction -->
-    <mu1>1</mu1>
-    <mu2>1</mu2>
+    <mu1>.1</mu1>
+    <mu2>.1</mu2>
   </gazebo>
   <!-- Add visual params -->

File: xacro/arduplane.xacro (robot description, xacro)
@@ -12,5 +12,5 @@
         -->
         <modelXYZToAirplaneXForwardZDown>0 0 0 0 0 0</modelXYZToAirplaneXForwardZDown>
-        <gazeboXYZToNED>0 0 0 3.141593 0 0</gazeboXYZToNED>
+        <gazeboXYZToNED>0 0 0 3.141593 0 1.57079</gazeboXYZToNED>
         <imuName>${ns}/imu_link::imu_sensor</imuName>
         <connectionTimeoutMaxCount>5</connectionTimeoutMaxCount>
@@ -18,9 +18,9 @@
           <type>VELOCITY</type>
           <offset>0</offset>
-          <p_gain>0</p_gain>
-          <i_gain>10</i_gain>
+          <p_gain>.1</p_gain>
+          <i_gain>0</i_gain>
           <d_gain>0</d_gain>
-          <i_max>100000</i_max>
-          <i_min>-100000</i_min>
+          <i_max>0</i_max>
+          <i_min>0</i_min>
           <cmd_max>2.5</cmd_max>
           <cmd_min>0</cmd_min>
@@ -32,5 +32,5 @@
           <type>POSITION</type>
           <offset>-0.5</offset>
-          <p_gain>0.20</p_gain>
+          <p_gain>2.00</p_gain>
           <i_gain>0</i_gain>
           <d_gain>1.50</d_gain>
@@ -46,5 +46,5 @@
           <type>POSITION</type>
           <offset>-0.5</offset>
-          <p_gain>0.20</p_gain>
+          <p_gain>2.00</p_gain>
           <i_gain>0</i_gain>
           <d_gain>1.50</d_gain>
@@ -60,5 +60,5 @@
           <type>POSITION</type>
           <offset>-0.5</offset>
-          <p_gain>0.20</p_gain>
+          <p_gain>2.00</p_gain>
           <i_gain>0</i_gain>
           <d_gain>1.50</d_gain>
@@ -74,5 +74,5 @@
           <type>POSITION</type>
           <offset>-0.5</offset>
-          <p_gain>0.20</p_gain>
+          <p_gain>2.00</p_gain>
           <i_gain>0</i_gain>
           <d_gain>1.50</d_gain>

File: xacro/plane_prop.xacro (robot description, xacro)
@@ -35,5 +35,5 @@
         <cma_stall>0</cma_stall>
         <cp>-0.37 0 0.77</cp>
-        <area>.001</area>
+        <area>.0001</area>
         <air_density>1.2041</air_density>
         <forward>0 -1 0</forward>
@@ -51,5 +51,5 @@
         <cma_stall>0</cma_stall>
         <cp>-0.37 0 -0.77</cp>
-        <area>.001</area>
+        <area>.0001</area>
         <air_density>1.2041</air_density>
         <forward>0 1 0</forward>
